File: hardware/v4_pcb_pilot/nanosun-pcb/nanosun-pcb.kicad_pcb (KiCad board)
At the start: 2 copper layers, 165 x 165 mm, 38 parts, among them J1 +12V, J2 DIN, J3 GND, J4 +5V, U1 MP1584EN_Module

Commit message: final checklists
Parts:
- added RPI_MH10: MountingHole_2.5mm, MountingHole:MountingHole_2.5mm, F.Cu at (131.5, 71.0)
- added RPI_MH7: MountingHole_2.5mm, MountingHole:MountingHole_2.5mm, F.Cu at (108.5, 71.0)
- added RPI_MH8: MountingHole_2.5mm, MountingHole:MountingHole_2.5mm, F.Cu at (131.5, 129.0)
- added RPI_MH9: MountingHole_2.5mm, MountingHole:MountingHole_2.5mm, F.Cu at (108.5, 129.0)
- moved 5V 18.7 mm to (150.0, 87.5)
- moved GND 13.5 mm to (150.0, 112.5)
- moved 12V 5.00 mm to (150.0, 125.0)
- renumbered J1 to 12V, J4 to 5V, J2 to DIN, J3 to GND, REF** to MH1, REF** to MH2, REF** to MH3, REF** to MH4, REF** to MH5, REF** to MH6
Routing:
- net GND: track 1536.0 -> 536.2 mm
- net +12V: track 1446.6 -> 533.2 mm
- net +5V: track 0.00 -> 44.7 mm
