File: hardware/v4_pcb_pilot/nanosun-pcb/nanosun-pcb.kicad_pcb (KiCad board)
At the start: 2 copper layers, 165 x 165 mm, 42 parts, among them U1 MP1584EN_Module

Commit message: pretty lines
Routing:
- net GND: track 536.2 -> 545.8 mm
- net Net-(LED5-DOUT): track 10.9 -> 14.2 mm
- net Net-(LED2-DOUT): track 17.2 -> 14.0 mm
- net Net-(LED10-DIN): track 14.1 -> 16.0 mm
- net +12V: track 533.2 -> 531.4 mm

Commit message: sent pcb for manufacturing
Parts:
- moved MH2 73.0 mm to (161.0, 40.0)
- moved MH3 72.9 mm to (161.0, 160.0)
- moved R1 40.0 mm to (115.1, 31.2)
- moved 12V 40.0 mm to (110.0, 125.0)
- moved 5V 40.0 mm to (110.0, 87.5)
- moved C1 40.0 mm to (111.8, 50.0)
- moved C2 40.0 mm to (111.8, 150.0)
- moved DIN 40.0 mm to (110.0, 75.0)
- moved GND 40.0 mm to (110.0, 112.5)
- moved LED1 40.0 mm to (91.2, 28.1)
- moved LED10 40.0 mm to (185.0, 84.3)
- moved LED11 40.0 mm to (35.0, 90.6)
- moved LED12 40.0 mm to (185.0, 96.8)
- moved LED13 40.0 mm to (35.0, 103.1)
- moved LED14 40.0 mm to (185.0, 109.3)
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Routing:
- net +12V: track 531.4 -> 586.2 mm
- net GND: track 545.8 -> 564.6 mm
- net Net-(LED1-DOUT): track 26.5 -> 21.3 mm
- net Net-(LED23-DOUT): track 26.5 -> 21.3 mm
- net Net-(LED10-DIN): track 16.0 -> 11.1 mm
- net Net-(LED2-DOUT): track 14.0 -> 10.9 mm
- net Net-(LED10-DOUT): track 9.71 -> 10.2 mm
Other:
- board text added: "digital sun nano v0"
- board text added: "© Simonas Sankauskas 2026"
