File: hardware/v4_pcb_pilot/nanosun-pcb/nanosun-pcb.kicad_sch (KiCad schematic)
At the start: 32 parts, among them J1 +12V, J2 DIN, J3 GND, J4 +5V, U1 MP1584EN_Module

Commit message: final checklists
Parts:
- renumbered J1 to 12V, J4 to 5V, J2 to DIN, J3 to GND
Changed lines of the file:
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@@
 		(on_board yes)
 		(dnp no)
-		(property "Reference" "J1"
+		(property "Reference" "12V"
 			(at 16.764 38.354 0)
 			(effects
@@
 			(project "nanosun-pcb"
 				(path "/9427757f-2137-44ed-ab82-f8a05bdcd89a"
-					(reference "J1")
+					(reference "12V")
 					(unit 1)
 				)
@@
 		(on_board yes)
 		(dnp no)
-		(property "Reference" "J2"
+		(property "Reference" "DIN"
 			(at 16.51 28.448 0)
 			(effects
@@
 			(project "nanosun-pcb"
 				(path "/9427757f-2137-44ed-ab82-f8a05bdcd89a"
-					(reference "J2")
+					(reference "DIN")
 					(unit 1)
 				)
@@
 		(on_board yes)
 		(dnp no)
-		(property "Reference" "J3"
+		(property "Reference" "GND"
 			(at 16.51 51.816 0)
 			(effects
@@
 			(project "nanosun-pcb"
 				(path "/9427757f-2137-44ed-ab82-f8a05bdcd89a"
-					(reference "J3")
+					(reference "GND")
 					(unit 1)
 				)
@@
 		(on_board yes)
 		(dnp no)
-		(property "Reference" "J4"
+		(property "Reference" "5V"
 			(at 110.236 161.29 0)
 			(effects
@@
 			(project "nanosun-pcb"
 				(path "/9427757f-2137-44ed-ab82-f8a05bdcd89a"
-					(reference "J4")
-					(unit 1)
-				)
+					(reference "5V")
+					(unit 1)
+				)
